File: STM_Morpho_Uno.kicad_pcb (KiCad board)
At the start: 2 copper layers, 70 x 59 mm, 6 parts, among them CN10 Conn_02x19_Odd_Even, CN5 Conn_01x10_Female, CN6 Conn_01x08_Female, CN7 Conn_02x19_Odd_Even, CN8 Conn_01x06_Female, CN9 Conn_01x08_Female

Commit message: fix, right uno connector where upside down compared to datasheet
Parts:
- moved CN5 22.9 mm to (189.1, 95.1), turned to 180 degrees
- moved CN9 17.8 mm to (189.1, 117.0), turned to 180 degrees
Connections:
- CN5 pad 1: Net-(CN10-Pad3) -> Net-(CN10-Pad21)
- CN5 pad 10: Net-(CN10-Pad21) -> Net-(CN10-Pad3)
- CN5 pad 2: Net-(CN10-Pad5) -> Net-(CN10-Pad19)
- CN5 pad 3: Net-(CN10-Pad7) -> Net-(CN10-Pad17)
- CN5 pad 4: Net-(CN10-Pad9) -> Net-(CN10-Pad15)
- CN5 pad 5: Net-(CN10-Pad11) -> Net-(CN10-Pad13)
- CN5 pad 6: Net-(CN10-Pad13) -> Net-(CN10-Pad11)
- CN5 pad 7: Net-(CN10-Pad15) -> Net-(CN10-Pad9)
- CN5 pad 8: Net-(CN10-Pad17) -> Net-(CN10-Pad7)
- CN5 pad 9: Net-(CN10-Pad19) -> Net-(CN10-Pad5)
- CN9 pad 1: Net-(CN10-Pad23) -> Net-(CN10-Pad37)
- CN9 pad 2: Net-(CN10-Pad25) -> Net-(CN10-Pad35)
- CN9 pad 3: Net-(CN10-Pad27) -> Net-(CN10-Pad33)
- CN9 pad 4: Net-(CN10-Pad29) -> Net-(CN10-Pad31)
- CN9 pad 5: Net-(CN10-Pad31) -> Net-(CN10-Pad29)
- CN9 pad 6: Net-(CN10-Pad33) -> Net-(CN10-Pad27)
- CN9 pad 7: Net-(CN10-Pad35) -> Net-(CN10-Pad25)
- CN9 pad 8: Net-(CN10-Pad37) -> Net-(CN10-Pad23)
